Commit message: integrating diff_drive ros2_control

File: description/urdf/ridgeback_ur5.urdf.xacro (robot description, xacro)
@@ -26,9 +26,4 @@
     <color rgba="0.15 0.15 0.15 1.0"/>
   </material>
-  <xacro:if value="$(arg ros2_control_mode)">
-    <link name="world"/>
-    <link name="base_x_link"/>
-    <link name="base_y_link"/>
-  </xacro:if>
   <link name="front_rocker_link">
     <visual>
@@ -173,27 +168,4 @@
   </joint>
   <link name="base_link"/>
-  <xacro:if value="$(arg ros2_control_mode)">
-    <joint name="base_x_joint" type="prismatic">
-      <origin rpy="0 0 0" xyz="0 0 0"/>
-      <parent link="world"/>
-      <child link="base_x_link"/>
-      <axis xyz="1 0 0"/>
-      <limit effort="1.0" lower="-1000" upper="1000" velocity="10"/>
-    </joint>
-    <joint name="base_y_joint" type="prismatic">
-      <origin rpy="0 0 0" xyz="0 0 0"/>
-      <parent link="base_x_link"/>
-      <child link="base_y_link"/>
-      <axis xyz="0 1 0"/>
-      <limit effort="1.0" lower="-1000" upper="1000" velocity="10"/>
-    </joint>
-    <joint name="base_yaw_joint" type="continuous">
-      <origin rpy="0 0 0" xyz="0 0 0"/>
-      <parent link="base_y_link"/>
-      <child link="base_link"/>
-      <axis xyz="0 0 1"/>
-      <limit effort="1.0" velocity="10"/>
-    </joint>
-  </xacro:if>
   <joint name="base_link_joint" type="fixed">
     <origin rpy="0 0 0" xyz="0 0 0"/>
@@ -691,18 +663,13 @@
         <state_interface name="velocity" />
       </joint>
-      <joint name="base_forward_joint">
-        <command_interface name="velocity" />
-        <state_interface name="velocity" />
-      </joint>
-      <joint name="base_yaw_joint">
-        <command_interface name="velocity" />
-        <state_interface name="position" />
-        <state_interface name="velocity" />
-      </joint>
-      <joint name="base_x_joint">
-        <state_interface name="position" />
-      </joint>
-      <joint name="base_y_joint">
-        <state_interface name="position" />
+      <joint name="left_wheel_joint">
+        <command_interface name="velocity" />
+        <state_interface name="position" />
+        <state_interface name="velocity" />
+      </joint>
+      <joint name="right_wheel_joint">
+        <command_interface name="velocity" />
+        <state_interface name="position" />
+        <state_interface name="velocity" />
       </joint>
     </ros2_control>
